File: microcontrollerinator.kicad_sch (KiCad schematic)
At the start: 45 parts, among them J1 USB_C_Receptacle_USB2.0_14P, J2 Conn_01x20, J3 Conn_01x20, J4 Conn_01x03, J5 Conn_01x03, Q1 AO3401A, SW1 SW_Push, U1 RP2040, U2 MCP1700x-330xxTT, U3 W25Q128JVS, U4 BQ21040DBV, Y1 12MHz

Commit message: routing pcb
Parts:
- removed BT1: Battery_Cell, symbol Device:Battery_Cell
- removed JP1: SolderJumper_2_Bridged, symbol Jumper:SolderJumper_2_Bridged
- added JP1: SolderJumper_2_Open, Jumper:SolderJumper-2_P1.3mm_Open_RoundedPad1.0x1.5mm, symbol Jumper:SolderJumper_2_Open
- added R11: 2K, Resistor_SMD:R_0402_1005Metric, symbol Device:R
- added R12: 7K, Resistor_SMD:R_0402_1005Metric, symbol Device:R
- C1, C10, C11, C12, C15, C16, C2, C3, C4, C5, C6, C7, C8, C9: footprint (none) -> Capacitor_SMD:C_0402_1005Metric
- C13, C14: footprint (none) -> Capacitor_SMD:C_0603_1608Metric
- C17, C18, C19: footprint (none) -> Capacitor_SMD:C_0504_1310Metric
- D1: footprint (none) -> Diode_SMD:D_0402_1005Metric
- D2: footprint (none) -> LED_SMD:LED_0603_1608Metric
- J1: footprint (none) -> Connector_USB:USB_C_Receptacle_HRO_TYPE-C-31-M-12
- J3: footprint (none) -> Connector_PinHeader_2.54mm:PinHeader_1x20_P2.54mm_Vertical
- R1, R10, R2, R3, R4, R5, R6, R7, R8, R9: footprint (none) -> Resistor_SMD:R_0402_1005Metric
- SW1: footprint (none) -> Button_Switch_SMD:SW_Push_SPST_NO_Alps_SKRK
- U3: footprint Package_SO:SOIC-8_5.3x5.3mm_P1.27mm -> Package_SON:Winbond_USON-8-1EP_3x2mm_P0.5mm_EP0.2x1.6mm
- Y1: footprint (none) -> Crystal:Crystal_SMD_3225-4Pin_3.2x2.5mm
Connections:
- net BAT_- is gone; now on net GND: J5.3 (Pin_3)
- net BAT_+: now also C19.1, Q1.3 (D), R8.1, U4.2 (OUT), R11.1
- net BAT_TS: now also JP1.2 (B)
- net GND: now also R12.2
- net GPIO23: now also J3.6 (Pin_6)
- net GPIO24: now also J3.4 (Pin_4)
- net GPIO29_ADC3: now also R11.2, R12.1; no longer J3.6 (Pin_6)
- net SWCLK: now also U1.24 (SWCLK)
- net SWD: now also U1.25 (SWD)
- net GPIO25: now reaches J3.2 (Pin_2)
- net GPIO25: now also U1.37 (GPIO25)
- net at R10.1: now also JP1.1 (A)
- no-connect marks 1 -> 0
Other:
- moved on the sheet: C18, C19, D2, Q1, R10, R3, R4, R8, R9, U1, U4

Commit message: finished routing pcb
Parts:
- C17, C18, C19: footprint Capacitor_SMD:C_0504_1310Metric -> Capacitor_SMD:C_0402_1005Metric
Changed lines of the file:
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@@
 			)
 		)
-		(property "Footprint" "Capacitor_SMD:C_0504_1310Metric"
+		(property "Footprint" "Capacitor_SMD:C_0402_1005Metric"
 			(at 201.6252 133.35 0)
 			(effects
@@
 			)
 		)
-		(property "Footprint" "Capacitor_SMD:C_0504_1310Metric"
+		(property "Footprint" "Capacitor_SMD:C_0402_1005Metric"
 			(at 267.97 30.7848 0)
 			(effects
@@
 			)
 		)
-		(property "Footprint" "Capacitor_SMD:C_0504_1310Metric"
+		(property "Footprint" "Capacitor_SMD:C_0402_1005Metric"
 			(at 248.6152 133.35 0)
 			(effects

Commit message: added production files
Parts:
- R11: value 2K -> 1K
- R12: value 7K -> 3.2K
Changed lines of the file:
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@@
 			)
 		)
-		(property "Value" "2K"
+		(property "Value" "1K"
 			(at 271.018 130.81 0)
 			(effects
@@
 			)
 		)
-		(property "Value" "7K"
+		(property "Value" "3.2K"
 			(at 271.018 140.97 0)
 			(effects
