File: microcontrollerinator.kicad_sch (KiCad schematic)
At the start: 46 parts, among them J1 USB_C_Receptacle_USB2.0_14P, J2 Conn_01x20, J3 Conn_01x20, J4 Conn_01x03, J5 Conn_01x03, Q1 AO3401A, SW1 SW_Push, U1 RP2040, U2 MCP1700x-330xxTT, U3 W25Q128JVS, U4 BQ21040DBV, Y1 12MHz

Commit message: fixed pcb
Parts:
- R3, R4: value 27K -> 27
Changed lines of the file:
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@@
 			)
 		)
-		(property "Value" "27K"
+		(property "Value" "27"
 			(at 115.57 76.962 90)
 			(effects
@@
 			)
 		)
-		(property "Value" "27K"
+		(property "Value" "27"
 			(at 115.57 70.358 90)
 			(effects
